Commit message: laser + config

File: urdf/mogi_bot.urdf (robot description, URDF)
Before this commit: robot mogi_bot, 6 links, 5 joints
Links:
- added link scan_link, mass 1e-5; collision box size=.1 .1 .1; visual mesh filename=package://assignment2/meshes/lidar.dae
Joints:
- added joint scan_joint: type fixed, parent base_link, child scan_link, origin xyz=0 0 0.15 rpy=0 0 0, axis 0 1 0
